Commit message: fix: separate planar odometry from elevated robot body

File: config/robot.urdf (robot description, URDF)
Before this commit: robot maintenance_robot, 6 links, 5 joints
Links:
- added link base_footprint
Joints:
- added joint body_height: type fixed, parent base_footprint, child base_link, origin xyz=0 0 .22
